File: pcba/spiflasher.sch (KiCad schematic (older format))
At the start: 41 parts, among them J1 USB_B_Micro, J2 Conn_02x04_Counter_Clockwise, J3 Conn_01x10, J4 Conn_01x10, U1 FT232H, U2 93LC56BT-I/OT, U3 TXB0104PW, Y1 12 MHz

Commit message: Changed crystal Digikey P/N to a non-marketplace one
Parts:
- Y1: Digikey 2388-SXT32420AA07-12.000M-ND -> XC2911CT-ND
Changed lines of the file:
@@
 F 3 "~" H 4250 4750 50  0001 C CNN
 F 4 "C9002" H 4250 4750 50  0001 C CNN "LCSC"
-F 5 " 2388-SXT32420AA07-12.000M-ND " H 4250 4750 50  0001 C CNN "Digikey"
+F 5 " XC2911CT-ND " H 4250 4750 50  0001 C CNN "Digikey"
 	1    4250 4750
 	0    1    1    0

Commit message: Removed unnecessary components.
Parts:
- removed C10, C8: 4.7u, Capacitor_SMD:C_0603_1608Metric, symbol Device:C_Small
- removed C15: 0.1u, Capacitor_SMD:C_0603_1608Metric, symbol Device:C_Small
- removed J3, J4: Conn_01x10, Connector_PinHeader_2.54mm:PinHeader_1x10_P2.54mm_Vertical, symbol Connector_Generic:Conn_01x10
- removed R3, R4, R5: 10k, Resistor_SMD:R_0603_1608Metric, symbol Device:R_Small_US
- removed R6: 2k, Resistor_SMD:R_0603_1608Metric, symbol Device:R_Small_US
- removed U2: 93LC56BT-I/OT, Package_TO_SOT_SMD:SOT-23-6, symbol Memory_EEPROM:93LCxxBxxOT
- Y1: footprint Crystal:Crystal_SMD_3225-4Pin_3.2x2.5mm_HandSoldering -> Crystal:Crystal_SMD_3225-4Pin_3.2x2.5mm
- renumbered C20 to C10, C3 to C11, C4 to C12, C5 to C13, C6 to C14, C7 to C15, C9 to C3, C11 to C4, C12 to C5, C13 to C6, C14 to C7, C18 to C8, C19 to C9, R7 to R1, R8 to R2, R9 to R3, R1 to R4, R2 to R5, U3 to U1, U1 to U2
Connections:
- no-connect marks 3 -> 18
Other:
- moved on the sheet: C1, C10, C11, C12, C13, C14, C15, C16, C17, C2, C3, C4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

Commit message: Low profile USB port. Final Rev 2
Parts:
- added NT1, NT2, NT3: Net-Tie_2, NetTie:NetTie-2_SMD_Pad0.5mm, symbol Device:Net-Tie_2
- C1, L1, L2, L3: Config (none) -> DNF
- J1: footprint Connector_USB:USB_Micro-B_Wuerth_629105150521 -> Local:USB_Micro-B_GCT_USB3070; Digikey 732-5960-1-ND -> 2073-USB3070-30-ACT-ND
Connections:
- net +3V3: now also NT2.1, NT3.1
- net VBUS: now also NT1.2
- net at C1.1, J1.1 (VBUS), L1.2: now also NT1.1
- net at C3.1, L2.1, U2.3 (VPHY): now also NT2.2
- net at C4.1, L3.1, U2.8 (VPLL): now also NT3.2
Changed lines of the file:
@@
 U 1 1 5F4F5F59
 P 3300 3250
-F 0 "L2" V 3119 3250 50  0000 C CNN
-F 1 "600R/0.5A" V 3210 3250 50  0000 C CNN
+F 0 "L2" V 3029 3250 50  0000 C CNN
+F 1 "600R/0.5A" V 3120 3250 50  0000 C CNN
 F 2 "Inductor_SMD:L_0603_1608Metric" H 3300 3250 50  0001 C CNN
 F 3 "~" H 3300 3250 50  0001 C CNN
 F 4 "C21189" H 3300 3250 50  0001 C CNN "LCSC"
 F 5 " 445-2205-1-ND " H 3300 3250 50  0001 C CNN "Digikey"
+F 6 "DNF" V 3211 3250 50  0000 C CNN "Config"
 	1    3300 3250
 	0    1    1    0
@@
 U 1 1 5F4F676C
 P 4200 3250
-F 0 "L3" V 4019 3250 50  0000 C CNN
-F 1 "600R/0.5A" V 4110 3250 50  0000 C CNN
+F 0 "L3" V 3900 3250 50  0000 C CNN
+F 1 "600R/0.5A" V 4000 3250 50  0000 C CNN
 F 2 "Inductor_SMD:L_0603_1608Metric" H 4200 3250 50  0001 C CNN
 F 3 "~" H 4200 3250 50  0001 C CNN
 F 4 "C21189" H 4200 3250 50  0001 C CNN "LCSC"
 F 5 " 445-2205-1-ND " H 4200 3250 50  0001 C CNN "Digikey"
+F 6 "DNF" V 4100 3250 50  0000 C CNN "Config"
 	1    4200 3250
 	0    1    1    0
 $EndComp
 Wire Wire Line
-	3050 3250 3200 3250
-Wire Wire Line
-	3950 3250 4100 3250
+	3050 3250 3150 3250
+Wire Wire Line
+	3950 3250 4050 3250
 Wire Wire Line
 	4800 3300 4950 3300
@@
 Wire Wire Line
 	2300 1250 2300 1600
-Wire Wire Line
-	2150 1250 2300 1250
-Wire Wire Line
-	1800 1250 1950 1250
-$Comp
-L Device:L_Core_Ferrite_Small L1
-U 1 1 5F4F53A2
-P 2050 1250
-F 0 "L1" V 1869 1250 50  0000 C CNN
-F 1 "600R/0.5A" V 1960 1250 50  0000 C CNN
-F 2 "Inductor_SMD:L_0603_1608Metric" H 2050 1250 50  0001 C CNN
-F 3 "~" H 2050 1250 50  0001 C CNN
-F 4 "C21189" H 2050 1250 50  0001 C CNN "LCSC"
-F 5 " 445-2205-1-ND " H 2050 1250 50  0001 C CNN "Digikey"
-	1    2050 1250
-	0    1    1    0
-$EndComp
 $Comp
 L Device:C_Small C2
@@
 U 1 1 5F4C72DC
 P 1800 1700
-F 0 "C1" H 1892 1746 50  0000 L CNN
-F 1 "10n" H 1892 1655 50  0000 L CNN
+F 0 "C1" H 1892 1791 50  0000 L CNN
+F 1 "10n" H 1892 1700 50  0000 L CNN
 F 2 "Capacitor_SMD:C_0603_1608Metric" H 1800 1700 50  0001 C CNN
 F 3 "~" H 1800 1700 50  0001 C CNN
 F 4 "C57112" H 1800 1700 50  0001 C CNN "LCSC"
+F 5 "DNF" H 1892 1609 50  0000 L CNN "Config"
 	1    1800 1700
 	1    0    0    -1
@@
 F 0 "J1" H 1207 1917 50  0000 C CNN
 F 1 "USB_B_Micro" H 1207 1826 50  0000 C CNN
-F 2 "Connector_USB:USB_Micro-B_Wuerth_629105150521" H 1300 1400 50  0001 C CNN
-F 3 "~" H 1300 1400 50  0001 C CNN
-F 4 " 732-5960-1-ND " H 1150 1450 50  0001 C CNN "Digikey"
+F 2 "Local:USB_Micro-B_GCT_USB3070" H 1300 1400 50  0001 C CNN
+F 3 "https://gct.co/files/drawings/usb3070.pdf" H 1300 1400 50  0001 C CNN
+F 4 "2073-USB3070-30-ACT-ND" H 1150 1450 50  0001 C CNN "Digikey"
 	1    1150 1450
 	1    0    0    -1
 $EndComp
 Wire Wire Line
-	4300 3250 4400 3250
+	4300 3250 4350 3250
 Connection ~ 4400 3250
 Wire Wire Line
@@
 	3800 3250 3800 3750
 Wire Wire Line
-	3400 3250 3500 3250
+	3400 3250 3450 3250
 Connection ~ 3500 3250
 Wire Wire Line
@@
 Wire Wire Line
 	3050 3700 3050 3650
+$Comp
+L Device:L_Core_Ferrite_Small L1
+U 1 1 5F4F53A2
+P 2050 1250
+F 0 "L1" V 1779 1250 50  0000 C CNN
+F 1 "600R/0.5A" V 1870 1250 50  0000 C CNN
+F 2 "Inductor_SMD:L_0603_1608Metric" H 2050 1250 50  0001 C CNN
+F 3 "~" H 2050 1250 50  0001 C CNN
+F 4 "C21189" H 2050 1250 50  0001 C CNN "LCSC"
+F 5 " 445-2205-1-ND " H 2050 1250 50  0001 C CNN "Digikey"
+F 6 "DNF" V 1961 1250 50  0000 C CNN "Config"
+	1    2050 1250
+	0    1    1    0
+$EndComp
+Wire Wire Line
+	3150 3250 3150 3200
+Wire Wire Line
+	3150 3200 3200 3200
+Wire Wire Line
+	3450 3200 3450 3250
+Connection ~ 3150 3250
+Wire Wire Line
+	3150 3250 3200 3250
+Connection ~ 3450 3250
+Wire Wire Line
+	3450 3250 3500 3250
+Wire Wire Line
+	4050 3250 4050 3200
+Wire Wire Line
+	4050 3200 4100 3200
+Wire Wire Line
+	4350 3200 4350 3250
+Connection ~ 4050 3250
+Wire Wire Line
+	4050 3250 4100 3250
+Connection ~ 4350 3250
+Wire Wire Line
+	4350 3250 4400 3250
+$Comp
+L Device:Net-Tie_2 NT2
+U 1 1 5F7824E6
+P 3300 3200
+F 0 "NT2" H 3300 3381 50  0001 C CNN
+F 1 "Net-Tie_2" H 3300 3290 50  0001 C CNN
+F 2 "NetTie:NetTie-2_SMD_Pad0.5mm" H 3300 3200 50  0001 C CNN
+F 3 "~" H 3300 3200 50  0001 C CNN
+	1    3300 3200
+	1    0    0    -1
+$EndComp
+Wire Wire Line
+	3400 3200 3450 3200
+$Comp
+L Device:Net-Tie_2 NT3
+U 1 1 5F7830CF
+P 4200 3200
+F 0 "NT3" H 4200 3381 50  0001 C CNN
+F 1 "Net-Tie_2" H 4200 3290 50  0001 C CNN
+F 2 "NetTie:NetTie-2_SMD_Pad0.5mm" H 4200 3200 50  0001 C CNN
+F 3 "~" H 4200 3200 50  0001 C CNN
+	1    4200 3200
+	1    0    0    -1
+$EndComp
+Wire Wire Line
+	4300 3200 4350 3200
+Wire Wire Line
+	2200 1250 2300 1250
+Wire Wire Line
+	2150 1250 2200 1250
+Connection ~ 2200 1250
+Wire Wire Line
+	2200 1200 2200 1250
+Wire Wire Line
+	2150 1200 2200 1200
+Wire Wire Line
+	1900 1250 1950 1250
+Wire Wire Line
+	1800 1250 1900 1250
+Connection ~ 1900 1250
+Wire Wire Line
+	1900 1250 1900 1200
+Wire Wire Line
+	1900 1200 1950 1200
+$Comp
+L Device:Net-Tie_2 NT1
+U 1 1 5F77BE96
+P 2050 1200
+F 0 "NT1" H 2050 1381 50  0001 C CNN
+F 1 "Net-Tie_2" H 2050 1290 50  0001 C CNN
+F 2 "NetTie:NetTie-2_SMD_Pad0.5mm" H 2050 1200 50  0001 C CNN
+F 3 "~" H 2050 1200 50  0001 C CNN
+	1    2050 1200
+	1    0    0    -1
+$EndComp
 $EndSCHEMATC
